File: SiNEDevBoard.sch (EAGLE design)
At the start: 33 parts, among them IC1 ATTINY24/44/84-SSU, IC2 74HC164D, J1 AVR_SPI_PRG_6NS

Commit message: DevBoard v0.2
Parts:
- added JP1, JP2, JP3: FIDUCIAL1X2.5-STOP, CISECO eaglecad designs:FIDUCIAL1X2.5-STOP
- added S1: (no value), CISECO eaglecad designs:TAC_SWITCHXINO_SMD
Changed lines of the file:
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@@
 <?xml version="1.0" encoding="utf-8"?>
 <!DOCTYPE eagle SYSTEM "eagle.dtd">
-<eagle version="6.2">
+<eagle version="6.1">
 <drawing>
 <settings>
@@
 <layers>
 <layer number="1" name="Top" color="4" fill="1" visible="no" active="no"/>
+<layer number="2" name="Route2" color="1" fill="3" visible="no" active="no"/>
+<layer number="3" name="Route3" color="4" fill="3" visible="no" active="no"/>
+<layer number="4" name="Route4" color="1" fill="4" visible="no" active="no"/>
+<layer number="5" name="Route5" color="4" fill="4" visible="no" active="no"/>
+<layer number="6" name="Route6" color="1" fill="8" visible="no" active="no"/>
+<layer number="7" name="Route7" color="4" fill="8" visible="no" active="no"/>
+<layer number="8" name="Route8" color="1" fill="2" visible="no" active="no"/>
+<layer number="9" name="Route9" color="4" fill="2" visible="no" active="no"/>
+<layer number="10" name="Route10" color="1" fill="7" visible="no" active="no"/>
+<layer number="11" name="Route11" color="4" fill="7" visible="no" active="no"/>
+<layer number="12" name="Route12" color="1" fill="5" visible="no" active="no"/>
+<layer number="13" name="Route13" color="4" fill="5" visible="no" active="no"/>
+<layer number="14" name="Route14" color="1" fill="6" visible="no" active="no"/>
+<layer number="15" name="Route15" color="4" fill="6" visible="no" active="no"/>
 <layer number="16" name="Bottom" color="1" fill="1" visible="no" active="no"/>
 <layer number="17" name="Pads" color="2" fill="1" visible="no" active="no"/>
@@
 <layer number="112" name="tSilk" color="7" fill="1" visible="yes" active="yes"/>
 <layer number="116" name="Patch_BOT" color="9" fill="4" visible="no" active="yes"/>
+<layer number="118" name="Rect_Pads" color="4" fill="1" visible="yes" active="yes"/>
+<layer number="120" name="120" color="7" fill="1" visible="yes" active="yes"/>
 <layer number="121" name="_tsilk" color="7" fill="1" visible="no" active="yes"/>
 <layer number="122" name="_bsilk" color="7" fill="1" visible="no" active="yes"/>
@@
 <part name="SJ1" library="SparkFun" deviceset="SOLDERJUMPER" device="TRACE"/>
 <part name="SJ2" library="SparkFun" deviceset="SOLDERJUMPER" device="TRACE"/>
+<part name="JP1" library="CISECO eaglecad designs" deviceset="FIDUCIAL" device="1X2.5-STOP"/>
+<part name="JP2" library="CISECO eaglecad designs" deviceset="FIDUCIAL" device="1X2.5-STOP"/>
+<part name="JP3" library="CISECO eaglecad designs" deviceset="FIDUCIAL" device="1X2.5-STOP"/>
+<part name="S1" library="CISECO eaglecad designs" deviceset="TAC_SWITCH" device="XINO_SMD"/>
 </parts>
 <sheets>
@@
 <instance part="P+2" gate="VCC" x="20.32" y="142.24" rot="R90"/>
 <instance part="BAT1" gate="G$1" x="86.36" y="114.3"/>
-<instance part="P+3" gate="VCC" x="78.74" y="114.3" rot="R90"/>
-<instance part="GND3" gate="1" x="93.98" y="114.3" rot="R90"/>
+<instance part="P+3" gate="VCC" x="76.2" y="114.3" rot="R90"/>
+<instance part="GND3" gate="1" x="96.52" y="114.3" rot="R90"/>
 <instance part="P+4" gate="VCC" x="27.94" y="99.06" rot="R180"/>
 <instance part="LED1" gate="G$1" x="195.58" y="162.56" rot="R90"/>
@@
 <instance part="SJ1" gate="1" x="68.58" y="40.64"/>
 <instance part="SJ2" gate="1" x="68.58" y="35.56"/>
+<instance part="JP1" gate="G$1" x="226.06" y="38.1"/>
+<instance part="JP2" gate="G$1" x="231.14" y="38.1"/>
+<instance part="JP3" gate="G$1" x="236.22" y="38.1"/>
+<instance part="S1" gate="S" x="149.86" y="81.28"/>
 </instances>
 <busses>
@@
 <pinref part="BAT1" gate="G$1" pin="-"/>
 <pinref part="GND3" gate="1" pin="GND"/>
+<wire x1="93.98" y1="114.3" x2="91.44" y2="114.3" width="0.1524" layer="91"/>
 </segment>
 <segment>
@@
 <pinref part="BAT1" gate="G$1" pin="+"/>
 <pinref part="P+3" gate="VCC" pin="VCC"/>
-</segment>
-<segment>
+<wire x1="78.74" y1="114.3" x2="81.28" y2="114.3" width="0.1524" layer="91"/>
+</segment>
+<segment>

Commit message: DevBoard V0.3
Parts:
- removed S1: (no value), CISECO eaglecad designs:TAC_SWITCHXINO_SMD
- C1: value (none) -> 0603 100nF
- R1, R2: value (none) -> 0603 10K
Other:
- moved on the sheet: R2
Changed lines of the file:
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@@
 <part name="GND1" library="supply1" deviceset="GND" device=""/>
 <part name="GND2" library="supply1" deviceset="GND" device=""/>
-<part name="R1" library="rcl" deviceset="R-EU_" device="R0805"/>
+<part name="R1" library="rcl" deviceset="R-EU_" device="R0805" value="0603 10K"/>
 <part name="P+1" library="supply1" deviceset="VCC" device=""/>
 <part name="P+2" library="supply1" deviceset="VCC" device=""/>
@@
 <part name="FRAME1" library="frames" deviceset="DINA4_L" device=""/>
 <part name="IC2" library="74xx-eu" deviceset="74*164" device="D" technology="HC"/>
-<part name="R2" library="rcl" deviceset="R-EU_" device="R0805"/>
+<part name="R2" library="rcl" deviceset="R-EU_" device="R0805" value="0603 10K"/>
 <part name="P+5" library="supply1" deviceset="VCC" device=""/>
 <part name="U$1" library="SparkFun" deviceset="IRRECEIVER" device="SMD"/>
 <part name="GND4" library="supply1" deviceset="GND" device=""/>
 <part name="P+6" library="supply1" deviceset="VCC" device=""/>
-<part name="C1" library="rcl" deviceset="C-EU" device="C0805"/>
+<part name="C1" library="rcl" deviceset="C-EU" device="C0805" value="0603 100nF"/>
 <part name="LED21" library="led" deviceset="LED" device="CHIPLED_1206"/>
 <part name="B1" library="microbuilder" deviceset="SWITCH_TACT_SMT" device=""/>
@@
 <part name="JP2" library="CISECO eaglecad designs" deviceset="FIDUCIAL" device="1X2.5-STOP"/>
 <part name="JP3" library="CISECO eaglecad designs" deviceset="FIDUCIAL" device="1X2.5-STOP"/>
-<part name="S1" library="CISECO eaglecad designs" deviceset="TAC_SWITCH" device="XINO_SMD"/>
 </parts>
 <sheets>
@@
 <instance part="FRAME1" gate="G$2" x="162.56" y="0"/>
 <instance part="IC2" gate="A" x="139.7" y="147.32"/>
-<instance part="R2" gate="G$1" x="121.92" y="152.4" rot="R180"/>
-<instance part="P+5" gate="VCC" x="114.3" y="152.4" rot="R90"/>
+<instance part="R2" gate="G$1" x="119.38" y="152.4" rot="R180"/>
+<instance part="P+5" gate="VCC" x="111.76" y="160.02"/>
 <instance part="U$1" gate="G$1" x="27.94" y="66.04"/>
 <instance part="GND4" gate="1" x="43.18" y="60.96" rot="R90"/>
-<instance part="P+6" gate="VCC" x="40.64" y="71.12" rot="R270"/>
+<instance part="P+6" gate="VCC" x="43.18" y="71.12" rot="R270"/>
 <instance part="C1" gate="G$1" x="48.26" y="68.58" rot="R90"/>
 <instance part="LED21" gate="G$1" x="99.06" y="66.04"/>
 <instance part="B1" gate="G$1" x="127" y="68.58"/>
 <instance part="B2" gate="G$1" x="127" y="86.36"/>
-<instance part="GND5" gate="1" x="134.62" y="86.36" rot="R90"/>
-<instance part="GND6" gate="1" x="134.62" y="68.58" rot="R90"/>
+<instance part="GND5" gate="1" x="137.16" y="86.36" rot="R90"/>
+<instance part="GND6" gate="1" x="137.16" y="68.58" rot="R90"/>
 <instance part="SJ1" gate="1" x="68.58" y="40.64"/>
 <instance part="SJ2" gate="1" x="68.58" y="35.56"/>
@@
 <instance part="JP2" gate="G$1" x="231.14" y="38.1"/>
 <instance part="JP3" gate="G$1" x="236.22" y="38.1"/>
-<instance part="S1" gate="S" x="149.86" y="81.28"/>
 </instances>
 <busses>
@@
 <pinref part="B2" gate="G$1" pin="S"/>
 <pinref part="GND5" gate="1" pin="GND"/>
+<wire x1="134.62" y1="86.36" x2="132.08" y2="86.36" width="0.1524" layer="91"/>
 </segment>
 <segment>
 <pinref part="B1" gate="G$1" pin="S"/>
 <pinref part="GND6" gate="1" pin="GND"/>
+<wire x1="134.62" y1="68.58" x2="132.08" y2="68.58" width="0.1524" layer="91"/>
 </segment>
 </net>
@@
 <segment>
 <pinref part="SJ1" gate="1" pin="2"/>
-<wire x1="73.66" y1="40.64" x2="81.28" y2="40.64" width="0.1524" layer="91"/>
-<label x="81.28" y="40.64" size="1.27" layer="95" xref="yes"/>
+<wire x1="73.66" y1="40.64" x2="96.52" y2="40.64" width="0.1524" layer="91"/>
+<label x="96.52" y="40.64" size="1.27" layer="95" xref="yes"/>
 </segment>
 </net>
@@
 <segment>
 <pinref part="SJ2" gate="1" pin="2"/>
-<wire x1="73.66" y1="35.56" x2="81.28" y2="35.56" width="0.1524" layer="91"/>
-<label x="81.28" y="35.56" size="1.27" layer="95" xref="yes"/>
+<wire x1="73.66" y1="35.56" x2="96.52" y2="35.56" width="0.1524" layer="91"/>
+<label x="96.52" y="35.56" size="1.27" layer="95" xref="yes"/>
 </segment>
 </net>
@@
 <pinref part="R2" gate="G$1" pin="2"/>
 <pinref part="P+5" gate="VCC" pin="VCC"/>
+<wire x1="111.76" y1="157.48" x2="111.76" y2="152.4" width="0.1524" layer="91"/>
+<wire x1="111.76" y1="152.4" x2="114.3" y2="152.4" width="0.1524" layer="91"/>
 </segment>
 <segment>
 <pinref part="U$1" gate="G$1" pin="VS"/>
 <pinref part="P+6" gate="VCC" pin="VCC"/>
+<wire x1="40.64" y1="71.12" x2="38.1" y2="71.12" width="0.1524" layer="91"/>
 </segment>
 </net>
@@
 <pinref part="IC2" gate="A" pin="B"/>
 <pinref part="R2" gate="G$1" pin="1"/>
-</segment>
-</net>
+<wire x1="124.46" y1="152.4" x2="127" y2="152.4" width="0.1524" layer="91"/>
+</segment>
+</net>

Commit message: DevBoard V0.4
Parts:
- removed U$1: IRRECEIVERSMD, SparkFun:IRRECEIVERSMD
- added TP1: TPB2,54, CISECO eaglecad designs:TPB2,54
- added U$2: IR-RECEIVER, CISECO eaglecad designs:IR-RECEIVER
Connections:
- removed net N$2: IC1.(PCINT10/INT0/OC0A/CKOUT)PB2
- new net TESTPAD: IC1.(PCINT10/INT0/OC0A/CKOUT)PB2, TP1.TP
- net GND: now also U$2.GND, U$2.NC/GND; no longer U$1.GND, U$1.GND1, U$1.GND2
- net N$6: now also U$2.OUT; no longer U$1.OUT
- net VCC: now also U$2.VS; no longer U$1.VS
Changed lines of the file:
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@@
 <part name="R2" library="rcl" deviceset="R-EU_" device="R0805" value="0603 10K"/>
 <part name="P+5" library="supply1" deviceset="VCC" device=""/>
-<part name="U$1" library="SparkFun" deviceset="IRRECEIVER" device="SMD"/>
-<part name="GND4" library="supply1" deviceset="GND" device=""/>
 <part name="P+6" library="supply1" deviceset="VCC" device=""/>
 <part name="C1" library="rcl" deviceset="C-EU" device="C0805" value="0603 100nF"/>
@@
 <part name="JP2" library="CISECO eaglecad designs" deviceset="FIDUCIAL" device="1X2.5-STOP"/>
 <part name="JP3" library="CISECO eaglecad designs" deviceset="FIDUCIAL" device="1X2.5-STOP"/>
+<part name="U$2" library="CISECO eaglecad designs" deviceset="IR-RECEIVER" device=""/>
+<part name="GND7" library="supply1" deviceset="GND" device=""/>
+<part name="TP1" library="CISECO eaglecad designs" deviceset="TP" device="B2,54"/>
 </parts>
 <sheets>
@@
 <instance part="R2" gate="G$1" x="119.38" y="152.4" rot="R180"/>
 <instance part="P+5" gate="VCC" x="111.76" y="160.02"/>
-<instance part="U$1" gate="G$1" x="27.94" y="66.04"/>
-<instance part="GND4" gate="1" x="43.18" y="60.96" rot="R90"/>
 <instance part="P+6" gate="VCC" x="43.18" y="71.12" rot="R270"/>
 <instance part="C1" gate="G$1" x="48.26" y="68.58" rot="R90"/>
@@
 <instance part="JP2" gate="G$1" x="231.14" y="38.1"/>
 <instance part="JP3" gate="G$1" x="236.22" y="38.1"/>
+<instance part="U$2" gate="G$1" x="22.86" y="73.66" rot="MR0"/>
+<instance part="GND7" gate="1" x="38.1" y="81.28" rot="R90"/>
+<instance part="TP1" gate="G$1" x="129.54" y="114.3"/>
 </instances>
 <busses>
@@
 </segment>
 <segment>
-<pinref part="U$1" gate="G$1" pin="GND2"/>
-<pinref part="GND4" gate="1" pin="GND"/>
-<wire x1="40.64" y1="60.96" x2="38.1" y2="60.96" width="0.1524" layer="91"/>
-<pinref part="U$1" gate="G$1" pin="GND"/>
-<wire x1="38.1" y1="66.04" x2="38.1" y2="63.5" width="0.1524" layer="91"/>
-<junction x="38.1" y="60.96"/>
-<pinref part="U$1" gate="G$1" pin="GND1"/>
-<junction x="38.1" y="63.5"/>
-<wire x1="38.1" y1="63.5" x2="38.1" y2="60.96" width="0.1524" layer="91"/>
-</segment>
-<segment>
 <pinref part="B2" gate="G$1" pin="S"/>
 <pinref part="GND5" gate="1" pin="GND"/>
@@
 <pinref part="GND6" gate="1" pin="GND"/>
 <wire x1="134.62" y1="68.58" x2="132.08" y2="68.58" width="0.1524" layer="91"/>
+</segment>
+<segment>
+<pinref part="U$2" gate="G$1" pin="NC/GND"/>
+<wire x1="30.48" y1="73.66" x2="33.02" y2="73.66" width="0.1524" layer="91"/>
+<wire x1="33.02" y1="73.66" x2="33.02" y2="76.2" width="0.1524" layer="91"/>
+<pinref part="U$2" gate="G$1" pin="GND"/>
+<wire x1="30.48" y1="76.2" x2="33.02" y2="76.2" width="0.1524" layer="91"/>
+<wire x1="33.02" y1="76.2" x2="33.02" y2="81.28" width="0.1524" layer="91"/>
+<wire x1="33.02" y1="81.28" x2="35.56" y2="81.28" width="0.1524" layer="91"/>
+<junction x="33.02" y="76.2"/>
+<pinref part="GND7" gate="1" pin="GND"/>
 </segment>
 </net>
@@
 </segment>
 </net>
-<net name="N$2" class="0">
-<segment>
-<pinref part="IC1" gate="1" pin="(PCINT10/INT0/OC0A/CKOUT)PB2"/>
-<wire x1="86.36" y1="157.48" x2="93.98" y2="157.48" width="0.1524" layer="91"/>
-<label x="93.98" y="157.48" size="1.27" layer="95" xref="yes"/>
-</segment>
-</net>
 <net name="VCC" class="0">
 <segment>
@@
 </segment>
 <segment>
-<pinref part="U$1" gate="G$1" pin="VS"/>
 <pinref part="P+6" gate="VCC" pin="VCC"/>
-<wire x1="40.64" y1="71.12" x2="38.1" y2="71.12" width="0.1524" layer="91"/>
+<wire x1="40.64" y1="71.12" x2="30.48" y2="71.12" width="0.1524" layer="91"/>
+<pinref part="U$2" gate="G$1" pin="VS"/>
 </segment>
 </net>
@@
 <net name="N$6" class="0">
 <segment>
-<pinref part="U$1" gate="G$1" pin="OUT"/>
 <pinref part="C1" gate="G$1" pin="1"/>
-<wire x1="45.72" y1="68.58" x2="38.1" y2="68.58" width="0.1524" layer="91"/>
+<wire x1="45.72" y1="68.58" x2="30.48" y2="68.58" width="0.1524" layer="91"/>
+<pinref part="U$2" gate="G$1" pin="OUT"/>
 </segment>
 </net>
@@
 </segment>
 </net>
+<net name="TESTPAD" class="0">
+<segment>
+<wire x1="127" y1="111.76" x2="129.54" y2="111.76" width="0.1524" layer="91"/>
+<label x="127" y="111.76" size="1.778" layer="95" rot="MR0" xref="yes"/>
+<pinref part="TP1" gate="G$1" pin="TP"/>
+</segment>
+<segment>
+<pinref part="IC1" gate="1" pin="(PCINT10/INT0/OC0A/CKOUT)PB2"/>
+<wire x1="86.36" y1="157.48" x2="93.98" y2="157.48" width="0.1524" layer="91"/>
+<label x="93.98" y="157.48" size="1.27" layer="95" xref="yes"/>
+</segment>
+</net>
