File: SiNEProduction.brd (EAGLE design)
At the start: 80 x 60 mm, 42 parts, among them IC1 74HCT164D, IC3 ATTINY24/44/84-SSU, J1 AVR_SPI_PRG_6NS

Commit message: Last tweaks for EMF Logo
Parts:
- added U$6: (no value), SiNE Parts:EMFLOGO
- U$2: value MINIEMF -> (none); device TiLDA:EMF-SMALL -> SiNE Parts:EMFLOGO1
- moved U$2 70.7 mm to (65.0, 42.0), flipped to the bottom
- moved BAT2 4.00 mm to (40.0, 26.0)
Routing:
- net GND: track 81.5 -> 85.5 mm
- net BTN2: track 82.0 -> 82.9 mm
Other:
- board text added: "Sponsored by:"
- board text added: "emfcamp.org/wave"
- board text removed: "Sunday 5th May 2013"
- board text removed: "www.emfcamp.org/wave"
Changed lines of the file:
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@@
 <layer number="22" name="bPlace" color="14" fill="1" visible="yes" active="yes"/>
 <layer number="23" name="tOrigins" color="15" fill="1" visible="yes" active="yes"/>
-<layer number="24" name="bOrigins" color="15" fill="1" visible="no" active="yes"/>
+<layer number="24" name="bOrigins" color="15" fill="1" visible="yes" active="yes"/>
 <layer number="25" name="tNames" color="7" fill="1" visible="no" active="yes"/>
 <layer number="26" name="bNames" color="7" fill="1" visible="no" active="yes"/>
 <layer number="27" name="tValues" color="7" fill="1" visible="no" active="yes"/>
 <layer number="28" name="bValues" color="7" fill="1" visible="no" active="yes"/>
-<layer number="29" name="tStop" color="7" fill="3" visible="no" active="yes"/>
+<layer number="29" name="tStop" color="7" fill="3" visible="yes" active="yes"/>
 <layer number="30" name="bStop" color="7" fill="6" visible="no" active="yes"/>
 <layer number="31" name="tCream" color="7" fill="4" visible="no" active="yes"/>
@@
 <layer number="40" name="bKeepout" color="1" fill="11" visible="no" active="yes"/>
 <layer number="41" name="tRestrict" color="4" fill="10" visible="no" active="yes"/>
-<layer number="42" name="bRestrict" color="1" fill="10" visible="no" active="yes"/>
+<layer number="42" name="bRestrict" color="1" fill="10" visible="yes" active="yes"/>
 <layer number="43" name="vRestrict" color="2" fill="10" visible="no" active="yes"/>
 <layer number="44" name="Drills" color="7" fill="1" visible="yes" active="yes"/>
@@
 <vertex x="70" y="13"/>
 </polygon>
-<circle x="40" y="22" radius="9" width="0" layer="42"/>
-<text x="62" y="41" size="2.54" layer="22" font="vector" ratio="15" rot="MR0">Electromagnetic Wave</text>
-<text x="62" y="38" size="2.54" layer="22" font="vector" ratio="15" rot="MR0">Sunday 5th May 2013</text>
-<text x="62" y="35" size="2.54" layer="22" font="vector" ratio="15" rot="MR0">www.emfcamp.org/wave</text>
-<text x="78" y="22" size="2.54" layer="22" font="vector" ratio="15" rot="MR0">Design by:</text>
-<text x="78" y="16" size="1.9304" layer="22" font="vector" ratio="15" rot="MR0">@CharlesYarnold</text>
-<text x="78" y="19" size="1.9304" layer="22" font="vector" ratio="15" rot="MR0">@thinkl33t</text>
-<text x="78" y="13" size="1.9304" layer="22" font="vector" ratio="15" rot="MR0">@dpslwk</text>
+<circle x="40" y="26" radius="9" width="0" layer="42"/>
+<text x="62" y="42" size="2.54" layer="22" font="vector" ratio="15" rot="MR0">Electromagnetic Wave</text>
+<text x="62" y="39" size="2.54" layer="22" font="vector" ratio="15" rot="MR0">emfcamp.org/wave</text>
+<text x="78" y="25" size="2.54" layer="22" font="vector" ratio="15" rot="MR0">Design by:</text>
+<text x="78" y="19" size="1.9304" layer="22" font="vector" ratio="15" rot="MR0">@CharlesYarnold</text>
+<text x="78" y="22" size="1.9304" layer="22" font="vector" ratio="15" rot="MR0">@thinkl33t</text>
+<text x="78" y="16" size="1.9304" layer="22" font="vector" ratio="15" rot="MR0">@dpslwk</text>
 <text x="22" y="22" size="2.54" layer="22" font="vector" ratio="15" rot="MR0">Built by:</text>
-<text x="49" y="51" size="6.4516" layer="22" font="vector" ratio="15" rot="MR0">SiNE</text>
+<text x="49" y="52" size="6.4516" layer="22" font="vector" ratio="15" rot="MR0">SiNE</text>
 <text x="15" y="7" size="1.778" layer="21" ratio="15">A</text>
 <text x="15" y="2" size="1.778" layer="21" ratio="15">K</text>
@@
 <text x="60" y="7" size="1.778" layer="21" ratio="15">J</text>
 <text x="60" y="2" size="1.778" layer="21" ratio="15">T</text>
+<text x="60" y="13" size="2.54" layer="22" font="vector" ratio="15" rot="MR0">Sponsored by:</text>
 </plain>
 <attributes>
@@
 <element name="SJ2" library="SparkFun" package="SJ_2S-TRACE" value="SOLDERJUMPERTRACE (NP)" x="76" y="21.5" rot="R270"/>
 <element name="IC3" library="SiNE Parts" package="SOIC14" value="ATTINY24/44/84-SSU" x="72" y="52" rot="R270"/>
-<element name="BAT2" library="SiNE Parts" package="BATTCON_20MM" value="" x="40" y="22" rot="MR180"/>
+<element name="BAT2" library="SiNE Parts" package="BATTCON_20MM" value="" x="40" y="26" rot="MR180"/>
 <element name="TP2" library="SiNE Parts" package="B2,54" value="TPB2,54" x="64" y="50">
 <attribute name="TP_SIGNAL_NAME" value="" x="79.24" y="-21.12" size="1.778" layer="27" display="off"/>
 </element>
 <element name="IC1" library="SiNE Parts" package="SO14" value="74HCT164D" x="10" y="51.5" rot="R270"/>
-<element name="U$2" library="TiLDA" package="EMF-SMALL" value="MINIEMF" x="6" y="3"/>
 <element name="U$3" library="SiNE Parts" package="TSOP-COMBINED" value="IR-RECEIVE-COMBINED" x="4.25" y="25" rot="R270"/>
 <element name="PAD1" library="wirepad" package="4,16O1,6" value="WIREPAD4,16O1,6" x="40" y="47.5"/>
@@
 <element name="JP2" library="CISECO eaglecad designs" package="FIDUCIAL-1X2.5-STOP" value="FIDUCIAL1X2.5-STOP" x="16" y="57"/>
 <element name="JP3" library="CISECO eaglecad designs" package="FIDUCIAL-1X2.5-STOP" value="FIDUCIAL1X2.5-STOP" x="3" y="11.3"/>
+<element name="U$6" library="SiNE Parts" package="EMFLOGO" value="" x="5.5" y="5.5"/>
+<element name="U$2" library="SiNE Parts" package="EMFLOGO1" value="" x="65" y="42" rot="MR0"/>
 </elements>
 <signals>
@@
 </polygon>
 <via x="2" y="8" extent="1-16" drill="0.6"/>
-<via x="5" y="8" extent="1-16" drill="0.6"/>
-<wire x1="2" y1="8" x2="5" y2="8" width="0.4064" layer="16"/>
+<via x="7" y="8" extent="1-16" drill="0.6"/>
+<wire x1="2" y1="8" x2="7" y2="8" width="0.4064" layer="16"/>
 <contactref element="B2" pad="B'"/>
 <contactref element="B1" pad="B'"/>
@@
 <wire x1="38" y1="12" x2="16" y2="12" width="0.6096" layer="16"/>
 <wire x1="16" y1="12" x2="12" y2="8" width="0.6096" layer="16"/>
-<wire x1="12" y1="8" x2="5" y2="8" width="0.6096" layer="16"/>
-<wire x1="40" y1="22" x2="40" y2="14" width="0.6096" layer="16"/>
+<wire x1="12" y1="8" x2="7" y2="8" width="0.6096" layer="16"/>
+<wire x1="40" y1="26" x2="40" y2="14" width="0.6096" layer="16"/>
 <wire x1="40" y1="14" x2="43" y2="11" width="0.6096" layer="16"/>
 <wire x1="43" y1="11" x2="63" y2="11" width="0.6096" layer="16"/>
@@
 <via x="15.5" y="47.5" extent="1-16" drill="0.6"/>
 <wire x1="15.5" y1="47.5" x2="15.5" y2="50" width="0.4064" layer="16"/>
-<wire x1="15.5" y1="50" x2="16.5" y2="51" width="0.4064" layer="16"/>
-<wire x1="16.5" y1="51" x2="58" y2="51" width="0.4064" layer="16"/>
-<wire x1="58" y1="51" x2="60" y2="53" width="0.4064" layer="16"/>
-<wire x1="60" y1="53" x2="77.5" y2="53" width="0.4064" layer="16"/>
+<wire x1="15.5" y1="50" x2="18.5" y2="53" width="0.4064" layer="16"/>
+<wire x1="18.5" y1="53" x2="77.5" y2="53" width="0.4064" layer="16"/>
 <wire x1="74.6035" y1="53.27" x2="77.23" y2="53.27" width="0.4064" layer="1"/>
 <wire x1="77.23" y1="53.27" x2="77.5" y2="53" width="0.4064" layer="1"/>
@@
 <via x="17" y="49" extent="1-16" drill="0.6"/>
 <wire x1="17" y1="49" x2="17" y2="49.5" width="0.4064" layer="16"/>
-<wire x1="17" y1="49.5" x2="17.5" y2="50" width="0.4064" layer="16"/>
-<wire x1="17.5" y1="50" x2="58.5" y2="50" width="0.4064" layer="16"/>
-<wire x1="58.5" y1="50" x2="60.5" y2="52" width="0.4064" layer="16"/>
-<wire x1="60.5" y1="52" x2="78.5" y2="52" width="0.4064" layer="16"/>
+<wire x1="17" y1="49.5" x2="19.5" y2="52" width="0.4064" layer="16"/>
+<wire x1="19.5" y1="52" x2="78.5" y2="52" width="0.4064" layer="16"/>
 <via x="78.5" y="52" extent="1-16" drill="0.6"/>
 <wire x1="78.5" y1="52" x2="74.6035" y2="52" width="0.4064" layer="1"/>
@@
 <via x="6" y="36" extent="1-16" drill="0.6"/>
 <wire x1="6" y1="36" x2="6" y2="49.5" width="0.4064" layer="16"/>
-<wire x1="6" y1="49.5" x2="10" y2="53.5" width="0.4064" layer="16"/>
-<wire x1="10" y1="53.5" x2="58.5" y2="53.5" width="0.4064" layer="16"/>
+<wire x1="6" y1="49.5" x2="11" y2="54.5" width="0.4064" layer="16"/>
+<wire x1="11" y1="54.5" x2="57.5" y2="54.5" width="0.4064" layer="16"/>
 <wire x1="69.3965" y1="53.27" x2="58.73" y2="53.27" width="0.4064" layer="1"/>
-<wire x1="58.73" y1="53.27" x2="58.5" y2="53.5" width="0.4064" layer="1"/>
-<via x="58.5" y="53.5" extent="1-16" drill="0.6"/>
+<wire x1="58.73" y1="53.27" x2="57.5" y2="54.5" width="0.4064" layer="1"/>
+<via x="57.5" y="54.5" extent="1-16" drill="0.6"/>
 </signal>
 <signal name="BTN1">
